Commit message: added visualization package

File: teleop_visualization/urdf/ring.urdf.xacro (robot description, xacro)
@@ -12,5 +12,5 @@
             <origin xyz="0.0 0.0 0.0" rpy="${pi/2} 0.0 0.0" />
             <geometry>
-                <mesh filename="file://$(find rviz_rings)/toroid.stl" scale="1.0 1.0 1.0" />
+                <mesh filename="file://$(find teleop_visualization)/toroid.stl" scale="1.0 1.0 1.0" />
             </geometry>
             <material name="Cyan">

Commit message: scaled rings

File: teleop_visualization/urdf/ring.urdf.xacro (robot description, xacro)
@@ -7,4 +7,10 @@
     <xacro:property name="orange" value="0.97 0.48 0.0 1.0" />
     <xacro:property name="red" value="0.88 0.0 0.06 1.0" />
+    <xacro:property name="white_scale" value="1.0 1.0 1.0" />
+    <xacro:property name="blue_scale" value="1.0 1.0 1.0" />
+    <xacro:property name="green_scale" value="0.93 1.0 0.93" />
+    <xacro:property name="yellow_scale" value="0.86 1.0 0.86" />
+    <xacro:property name="orange_scale" value="0.8 1.0 0.8" />
+    <xacro:property name="red_scale" value="0.75 1.0 0.75" />
     <!-- Base Link -->
     <link name="center">
@@ -12,5 +18,5 @@
             <origin xyz="0.0 0.0 0.0" rpy="${pi/2} 0.0 0.0" />
             <geometry>
-                <mesh filename="file://$(find teleop_visualization)/toroid.stl" scale="1.0 1.0 1.0" />
+                <mesh filename="file://$(find teleop_visualization)/measured_ring.stl" scale="${$(arg ring_color)_scale}" />
             </geometry>
             <material name="Cyan">

Commit message: minor cleanup

File: teleop_visualization/urdf/ring.urdf.xacro (robot description, xacro)
@@ -18,5 +18,5 @@
             <origin xyz="0.0 0.0 0.0" rpy="${pi/2} 0.0 0.0" />
             <geometry>
-                <mesh filename="file://$(find teleop_visualization)/measured_ring.stl" scale="${$(arg ring_color)_scale}" />
+                <mesh filename="file://$(find teleop_visualization)/ring.stl" scale="${$(arg ring_color)_scale}" />
             </geometry>
             <material name="Cyan">
