Commit message: Mapped haptx finger joints to "robot" finger joints

File: teleop_tasks/urdf/leftHand.gazebo.xacro (robot description, xacro)
@@ -1,11 +1,30 @@
 <?xml version="1.0"?>
 <robot xmlns:xacro="http://www.ros.org/wiki/xacro">
-    <!-- prevent gazebo from merging frames with fixed joints-->
+    <ros2_control name="GazeboSimSystem" type="system">
+        <hardware>
+            <plugin>gz_ros2_control/GazeboSimSystem</plugin>
+        </hardware>
+        <joint name="palm_x">
+            <command_interface name="position">
+                <param name="min">-1000</param>
+                <param name="max">1000</param>
+            </command_interface>
+            <state_interface name="position">
+                <param name="initial_value">0.0</param>
+            </state_interface>
+        </joint>
+    </ros2_control>
     <gazebo>
-        <plugin
+        <!-- <plugin
             filename="libignition-gazebo-joint-state-publisher-system.so"
             name="ignition::gazebo::systems::JointStatePublisher">
             <topic>/left_hand/joint_states</topic>
-        </plugin>
+        </plugin> -->
+        <!-- Joint state publisher -->
+        <!-- <plugin filename="libgz_ros2_control-system.so" name="gz_ros2_control::GazeboSimROS2ControlPlugin">
+            <robot_param>left_hand/robot_description</robot_param>
+            <robot_param_node>robot_state_publisher</robot_param_node>
+            <parameters>$(find teleop_tasks)/config/left_hand_controller.yaml</parameters>
+        </plugin> -->
     </gazebo>
 </robot>

Commit message: Created a launch file that just displays the left hand and no gazebo world

File: teleop_tasks/urdf/leftHand.gazebo.xacro (robot description, xacro)
@@ -1,30 +1,3 @@
 <?xml version="1.0"?>
 <robot xmlns:xacro="http://www.ros.org/wiki/xacro">
-    <ros2_control name="GazeboSimSystem" type="system">
-        <hardware>
-            <plugin>gz_ros2_control/GazeboSimSystem</plugin>
-        </hardware>
-        <joint name="palm_x">
-            <command_interface name="position">
-                <param name="min">-1000</param>
-                <param name="max">1000</param>
-            </command_interface>
-            <state_interface name="position">
-                <param name="initial_value">0.0</param>
-            </state_interface>
-        </joint>
-    </ros2_control>
-    <gazebo>
-        <!-- <plugin
-            filename="libignition-gazebo-joint-state-publisher-system.so"
-            name="ignition::gazebo::systems::JointStatePublisher">
-            <topic>/left_hand/joint_states</topic>
-        </plugin> -->
-        <!-- Joint state publisher -->
-        <!-- <plugin filename="libgz_ros2_control-system.so" name="gz_ros2_control::GazeboSimROS2ControlPlugin">
-            <robot_param>left_hand/robot_description</robot_param>
-            <robot_param_node>robot_state_publisher</robot_param_node>
-            <parameters>$(find teleop_tasks)/config/left_hand_controller.yaml</parameters>
-        </plugin> -->
-    </gazebo>
 </robot>

File: teleop_tasks/urdf/leftHand.urdf.xacro (robot description, xacro)
@@ -339,4 +339,4 @@
         </sensor>
     </gazebo>
-    <xacro:include filename="$(find teleop_tasks)/urdf/leftHand.gazebo.xacro"/>
+    <!-- <xacro:include filename="$(find teleop_tasks)/urdf/leftHand.gazebo.xacro"/> -->
 </robot>
