Commit message: Finished the left hand xacro

File: teleop_tasks/urdf/leftHand.urdf.xacro (robot description, xacro)
@@ -13,4 +13,74 @@
         </visual>
     </link>
+    <!-- World links that are needed to get a 6dof joint from world to palm -->
+    <xacro:macro name="dummy_world" params="num">
+        <link name="world_${num}">
+            <inertial>
+                <mass value="0.00001" />
+                <inertia
+                    ixx="${(1/12)*0.00001*(0.6**2 + 0.2**2)}"
+                    ixy="0.0"
+                    ixz="0.0"
+                    iyy="${(1/12)*0.00001*(2.5**2 + 0.2**2)}"
+                    iyz="0.0"
+                    izz="${(1/12)*0.00001*(0.6**2 + 2.5**2)}"
+                />
+            </inertial>
+            <visual>
+                <origin xyz="0 0 0.0" />
+                <geometry>
+                    <sphere radius="0.5"/>
+                </geometry>
+                <material name="">
+                    <color rgba="0 1 0 0" />
+                </material>
+            </visual>
+        </link>
+    </xacro:macro>
+    <xacro:dummy_world num="2"/>
+    <xacro:dummy_world num="3"/>
+    <xacro:dummy_world num="4"/>
+    <xacro:dummy_world num="5"/>
+    <xacro:dummy_world num="6"/>
+    <!-- World joints from world to palm -->
+    <joint name="palm_x" type="prismatic">
+        <origin xyz="0.0 0.0 0.0" rpy="0.0 0.0 0.0"/>
+        <parent link="world"/>
+        <child link="world_2"/>
+        <axis xyz="1.0 0.0 0.0"/>
+        <limit effort="30" velocity="1.0" lower="-10.0" upper="10.0"/>
+    </joint>
+    <joint name="palm_y" type="prismatic">
+        <origin xyz="0.0 0.0 0.0" rpy="0.0 0.0 0.0" />
+        <parent link="world_2"/>
+        <child link="world_3"/>
+        <axis xyz="0.0 1.0 0.0"/>
+        <limit effort="30" velocity="1.0" lower="-10.0" upper="10.0"/>
+    </joint>
+    <joint name="palm_z" type="prismatic">
+        <origin xyz="0.0 0.0 0.0" rpy="0.0 0.0 0.0" />
+        <parent link="world_3"/>
+        <child link="world_4"/>
+        <axis xyz="0.0 0.0 1.0"/>
+        <limit effort="30" velocity="1.0" lower="-10.0" upper="10.0"/>
+    </joint>
+    <joint name="palm_roll" type="continuous">
+        <origin xyz="0.0 0.0 0.0" rpy="0.0 0.0 0.0" />
+        <parent link="world_4"/>
+        <child link="world_5"/>
+        <axis xyz="1.0 0.0 0.0"/>
+    </joint>
+    <joint name="palm_pitch" type="continuous">
+        <origin xyz="0.0 0.0 0.0" rpy="0.0 0.0 0.0" />
+        <parent link="world_5"/>
+        <child link="world_6"/>
+        <axis xyz="0.0 1.0 0.0"/>
+    </joint>
+    <joint name="palm_yaw" type="continuous">
+        <origin xyz="0.0 0.0 0.0" rpy="0.0 0.0 0.0" />
+        <parent link="world_6"/>
+        <child link="palm"/>
+        <axis xyz="0.0 0.0 1.0"/>
+    </joint>
     <!-- The palm -->
     <link name="palm">
@@ -27,7 +97,7 @@
         </inertial>
         <visual>
-            <origin xyz="0 0 -0.5" />
+            <origin xyz="0 0 -0.0127" />
             <geometry>
-                <box size="5.0 5.0 1.0" />
+                <box size="0.0889 0.0889 0.0254" />
             </geometry>
             <material name="">
@@ -36,16 +106,10 @@
         </visual>
         <collision>
-            <origin xyz="0 0 -0.5" />
+            <origin xyz="0 0 -0.0127" />
             <geometry>
-                <box size="5.0 5.0 2.0" />
+                <box size="0.0889 0.0889 0.0254" />
             </geometry>
         </collision>
     </link>
-    <!-- World to palm joints -->
-    <joint name="world_palm" type="floating">
-        <origin xyz="0.0 0.0 0.0" rpy="0.0 0.0 0.0" />
-        <parent link="world"/>
-        <child link="palm"/>
-    </joint>
     <!-- Macro for the fingers -->
     <xacro:macro name="finger" params="name length color">
@@ -65,5 +129,5 @@
                 <origin xyz="${length/2} 0 0" />
                 <geometry>
-                    <box size="${length} 1.0 1.0"/>
+                    <box size="${length} 0.01905 0.01905"/>
                 </geometry>
                 <material name="">
@@ -74,5 +138,5 @@
                 <origin xyz="${length/2} 0 0" />
                 <geometry>
-                    <box size="${length} 1.0 1.0"/>
+                    <box size="${length} 0.01905 0.01905"/>
                 </geometry>
             </collision>
@@ -81,26 +145,26 @@
     <!-- Creating each finger -->
     <xacro:finger name="index_dumb" length="0.0001" color="0 0 0 0"/>
-    <xacro:finger name="index_1" length="${5.0/3}" color="1 0 0 1"/>
-    <xacro:finger name="index_2" length="${5.0/3}" color="0 1 0 1"/>
-    <xacro:finger name="index_3" length="${5.0/3}" color="0 0 1 1"/>
+    <xacro:finger name="index_1" length="${0.0762/3}" color="1 0 0 1"/>
+    <xacro:finger name="index_2" length="${0.0762/3}" color="0 1 0 1"/>
+    <xacro:finger name="index_3" length="${0.0762/3}" color="0 0 1 1"/>
     <xacro:finger name="index_tip" length="0.0001" color="0 0 0 0"/>
     <xacro:finger name="middle_dumb" length="0.0001" color="0 0 0 0"/>
-    <xacro:finger name="middle_1" length="${5.0/3}" color="1 0 0 1"/>
-    <xacro:finger name="middle_2" length="${5.0/3}" color="0 1 0 1"/>
-    <xacro:finger name="middle_3" length="${5.0/3}" color="0 0 1 1"/>
+    <xacro:finger name="middle_1" length="${0.0889/3}" color="1 0 0 1"/>
+    <xacro:finger name="middle_2" length="${0.0889/3}" color="0 1 0 1"/>
+    <xacro:finger name="middle_3" length="${0.0889/3}" color="0 0 1 1"/>
     <xacro:finger name="middle_tip" length="0.0001" color="0 0 0 0"/>
     <xacro:finger name="ring_dumb" length="0.0001" color="0 0 0 0"/>
-    <xacro:finger name="ring_1" length="${5.0/3}" color="1 0 0 1"/>
-    <xacro:finger name="ring_2" length="${5.0/3}" color="0 1 0 1"/>
-    <xacro:finger name="ring_3" length="${5.0/3}" color="0 0 1 1"/>
+    <xacro:finger name="ring_1" length="${0.0762/3}" color="1 0 0 1"/>
+    <xacro:finger name="ring_2" length="${0.0762/3}" color="0 1 0 1"/>
+    <xacro:finger name="ring_3" length="${0.0762/3}" color="0 0 1 1"/>
     <xacro:finger name="ring_tip" length="0.0001" color="0 0 0 0"/>
     <xacro:finger name="pinky_dumb" length="0.0001" color="0 0 0 0"/>
-    <xacro:finger name="pinky_1" length="1.0" color="1 0 0 1"/>
-    <xacro:finger name="pinky_2" length="1.0" color="0 1 0 1"/>
-    <xacro:finger name="pinky_3" length="1.0" color="0 0 1 1"/>
+    <xacro:finger name="pinky_1" length="${0.0635/3}" color="1 0 0 1"/>
+    <xacro:finger name="pinky_2" length="${0.0635/3}" color="0 1 0 1"/>
+    <xacro:finger name="pinky_3" length="${0.0635/3}" color="0 0 1 1"/>
     <xacro:finger name="pinky_tip" length="0.0001" color="0 0 0 0"/>
     <xacro:finger name="thumb_dumb" length="0.0001" color="0 0 0 0"/>
-    <xacro:finger name="thumb_1" length="1.5" color="1 0 0 1"/>
-    <xacro:finger name="thumb_2" length="1.5" color="0 1 0 1"/>
+    <xacro:finger name="thumb_1" length="${0.0635/2}" color="1 0 0 1"/>
+    <xacro:finger name="thumb_2" length="${0.0635/2}" color="0 1 0 1"/>
     <xacro:finger name="thumb_tip" length="0.0001" color="0 0 0 0"/>
     <!-- Finger joint macro -->
@@ -116,5 +180,5 @@
     <xacro:macro name="fingertip_joint" params="parent child length">
         <joint name="${parent}_${child}" type="fixed">
-            <origin xyz="${length/2} 0.0 0.5" rpy="0.0 0.0 0.0" />
+            <origin xyz="${length/2} 0.0 0.009525" rpy="0.0 0.0 0.0" />
             <parent link="${parent}"/>
             <child link="${child}"/>
@@ -123,5 +187,5 @@
     <!-- Thumb joints -->
     <joint name="palm_thumb_dumb" type="continuous">
-        <origin xyz="0.0 2.5 -0.5" rpy="0.0 0.0 ${radians(90.0)}" />
+        <origin xyz="0.0 0.04445 -0.009525" rpy="0.0 0.0 ${radians(90.0)}" />
         <axis xyz="0.0 0.0 1.0"/>
         <parent link="palm"/>
@@ -129,13 +193,9 @@
     </joint>
     <xacro:finger_joint parent="thumb_dumb" child="thumb_1" length="0.0"/>
-    <xacro:finger_joint parent="thumb_1" child="thumb_2" length="1.5"/>
-    <joint name="thumb_2_thumb_tip" type="fixed">
-            <origin xyz="0.75 0.0 0.5" rpy="0.0 0.0 ${radians(-90.0)}" />
-            <parent link="thumb_2"/>
-            <child link="thumb_tip"/>
-    </joint>
+    <xacro:finger_joint parent="thumb_1" child="thumb_2" length="${0.0635/2}"/>
+    <xacro:fingertip_joint parent="thumb_2" child="thumb_tip" length="${0.0635/2}"/>
     <!-- Index finger joints -->
     <joint name="palm_index_dumb" type="continuous">
-        <origin xyz="2.5 2.0 -0.5" rpy="0.0 0.0 0.0" />
+        <origin xyz="0.04445 0.03556 -0.009525" rpy="0.0 0.0 0.0" />
         <axis xyz="0.0 0.0 1.0"/>
         <parent link="palm"/>
@@ -143,10 +203,10 @@
     </joint>
     <xacro:finger_joint parent="index_dumb" child="index_1" length="0.0"/>
-    <xacro:finger_joint parent="index_1" child="index_2" length="${5.0/3}"/>
-    <xacro:finger_joint parent="index_2" child="index_3" length="${5.0/3}"/>
-    <xacro:fingertip_joint parent="index_3" child="index_tip" length="${5.0/3}"/>
+    <xacro:finger_joint parent="index_1" child="index_2" length="${0.0762/3}"/>
+    <xacro:finger_joint parent="index_2" child="index_3" length="${0.0762/3}"/>
+    <xacro:fingertip_joint parent="index_3" child="index_tip" length="${0.0762/3}"/>
     <!-- Middle finger joints -->
     <joint name="palm_middle_dumb" type="continuous">
-        <origin xyz="2.5 0.675 -0.5" rpy="0.0 0.0 0.0" />
+        <origin xyz="0.04445 0.0120015 -0.009525" rpy="0.0 0.0 0.0" />
         <axis xyz="0.0 0.0 1.0"/>
         <parent link="palm"/>
@@ -154,10 +214,10 @@
     </joint>
     <xacro:finger_joint parent="middle_dumb" child="middle_1" length="0.0"/>
-    <xacro:finger_joint parent="middle_1" child="middle_2" length="${5.0/3}"/>
-    <xacro:finger_joint parent="middle_2" child="middle_3" length="${5.0/3}"/>
-    <xacro:fingertip_joint parent="middle_3" child="middle_tip" length="${5.0/3}"/>
+    <xacro:finger_joint parent="middle_1" child="middle_2" length="${0.0889/3}"/>
+    <xacro:finger_joint parent="middle_2" child="middle_3" length="${0.0889/3}"/>
+    <xacro:fingertip_joint parent="middle_3" child="middle_tip" length="${0.0889/3}"/>
     <!-- Ring finger joints -->
     <joint name="palm_ring_dumb" type="continuous">
-        <origin xyz="2.5 -0.675 -0.5" rpy="0.0 0.0 0.0" />
+        <origin xyz="0.04445 -0.0120015 -0.009525" rpy="0.0 0.0 0.0" />
         <axis xyz="0.0 0.0 1.0"/>
         <parent link="palm"/>
@@ -165,10 +225,10 @@
     </joint>
     <xacro:finger_joint parent="ring_dumb" child="ring_1" length="0.0"/>
-    <xacro:finger_joint parent="ring_1" child="ring_2" length="${5.0/3}"/>
-    <xacro:finger_joint parent="ring_2" child="ring_3" length="${5.0/3}"/>
-    <xacro:fingertip_joint parent="ring_3" child="ring_tip" length="${5.0/3}"/>
+    <xacro:finger_joint parent="ring_1" child="ring_2" length="${0.0762/3}"/>
+    <xacro:finger_joint parent="ring_2" child="ring_3" length="${0.0762/3}"/>
+    <xacro:fingertip_joint parent="ring_3" child="ring_tip" length="${0.0762/3}"/>
     <!-- Pinky finger joints -->
     <joint name="palm_pinky_dumb" type="continuous">
-        <origin xyz="2.5 -2.0 -0.5" rpy="0.0 0.0 0.0" />
+        <origin xyz="0.04445 -0.03556 -0.009525" rpy="0.0 0.0 0.0" />
         <axis xyz="0.0 0.0 1.0"/>
         <parent link="palm"/>
@@ -176,8 +236,8 @@
     </joint>
     <xacro:finger_joint parent="pinky_dumb" child="pinky_1" length="0.0"/>
-    <xacro:finger_joint parent="pinky_1" child="pinky_2" length="1.0"/>
-    <xacro:finger_joint parent="pinky_2" child="pinky_3" length="1.0"/>
-    <xacro:fingertip_joint parent="pinky_3" child="pinky_tip" length="1.0"/>
-    <!-- Gazebo force macro -->
+    <xacro:finger_joint parent="pinky_1" child="pinky_2" length="${0.0635/3}"/>
+    <xacro:finger_joint parent="pinky_2" child="pinky_3" length="${0.0635/3}"/>
+    <xacro:fingertip_joint parent="pinky_3" child="pinky_tip" length="${0.0635/3}"/>
+    <!-- Gazebo contact force objects -->
     <gazebo reference="thumb_2_thumb_tip">
         <provideFeedback>true</provideFeedback>
@@ -195,5 +255,5 @@
         </sensor>
     </gazebo>
-    <gazebo reference="index_3_index_tip">
+    <!-- <gazebo reference="index_3_index_tip">
         <provideFeedback>true</provideFeedback>
         <preserveFixedJoint>true</preserveFixedJoint>
@@ -254,4 +314,4 @@
         </force_torque>
         </sensor>
-    </gazebo>
+    </gazebo> -->
 </robot>
